Commit message: Adding gripper URDFs and controller
* added 2f gripper controller

* added gripper controller

File: robo_gym/data/ur5/ur5_2f.urdf (robot description, URDF)
Before this commit: robot ur5, 20 links, 19 joints
Links:
- removed link tool0
- added link left_finger_pad; collision box size=0.0067 0.027 0.065; visual box size=0.0067 0.027 0.065
- added link right_finger_pad; collision box size=0.0067 0.027 0.065; visual box size=0.0067 0.027 0.065
Joints:
- removed joint finger_joint
- removed joint ur5_ee_gripper_joint
- removed joint wrist_3_link-tool0_fixed_joint
- added joint left_finger_pad_joint: type fixed, parent left_inner_finger, child left_finger_pad, origin xyz=0 0.0405 -0.02758 rpy=1.57 1.57 0
- added joint left_outer_knuckle_joint: type revolute, parent robotiq_arg2f_base_link, child left_outer_knuckle, origin xyz=0 -0.030601 0.054905 rpy=2.29579632679 0 0, axis -1 0 0, limit lower=0 upper=0.775 effort=1000 velocity=2.0
- added joint right_finger_pad_joint: type fixed, parent right_inner_finger, child right_finger_pad, origin xyz=0 0.0405 -0.02758 rpy=1.57 1.57 0
- added joint wrist_3_link-gripper_base_fixed_joint: type fixed, parent wrist_3_link, child robotiq_arg2f_base_link, origin xyz=0 0.0823 0 rpy=-1.57079632679 0 0
- joint left_inner_finger_joint: mimic joint=finger_joint multiplier=1 offset=0 -> joint=left_outer_knuckle_joint multiplier=1 offset=0
- joint left_inner_knuckle_joint: axis 1 0 0 -> -1 0 0; mimic joint=finger_joint multiplier=-1 offset=0 -> joint=left_outer_knuckle_joint multiplier=-1 offset=0
- joint right_inner_finger_joint: mimic joint=finger_joint multiplier=1 offset=0 -> joint=left_outer_knuckle_joint multiplier=1 offset=0
- joint right_inner_knuckle_joint: axis 1 0 0 -> -1 0 0; mimic joint=finger_joint multiplier=-1 offset=0 -> joint=left_outer_knuckle_joint multiplier=-1 offset=0
- joint right_outer_knuckle_joint: axis 1 0 0 -> -1 0 0; mimic joint=finger_joint multiplier=-1 offset=0 -> joint=left_outer_knuckle_joint multiplier=-1 offset=0

Commit message: Gripper stuff (#10)
* added 2f gripper controller

* added gripper controller

* refactored controllers and added controller interface

* Added randomization addon

* Created 3f controller and modified domain_randomization to download textures if not available

* removed textures dataset

* modified gitignore to ignore texture dataset

* Modified to download textures for user if they don't have it already

* Added comments and added back some commands and addons

* Separated randomization into visual and dynamics. Created an interface for the randomizers. Modified addon.py to accomodate for randomizer changes.

* Modified yaml for randomization

* removed domain_randomization

File: robo_gym/data/ur5/ur5_2f.urdf (robot description, URDF)
Before this commit: robot ur5, 21 links, 20 joints
Joints:
- joint left_outer_knuckle_joint: limit lower=0 upper=0.775 effort=1000 velocity=2.0 -> lower=0 upper=0.76 effort=1000 velocity=2.0

File: robo_gym/data/ur5/ur5_3f.urdf (robot description, URDF)
Before this commit: robot ur5, 25 links, 24 joints
Links:
- removed link tool0
- removed link tool1
Joints:
- removed joint palm_tool1
- removed joint ur5_ee_gripper_joint
- joint wrist_3_link-tool0_fixed_joint: child tool0 -> palm; origin xyz=0 0.0823 0 rpy=-1.57079632679 0 0 -> xyz=0 0.0823 0 rpy=0.0 0 0

Commit message: Gripper env (#16)
* added new addon to detect where an object is

* Created a pick and place env for the ur5. Modified controllers to take
position targets and changed position gains for smoother movements.

* Created distance reward and sensors

* last minute updates. Fixed some bugs when flattening state and action space and another in draw_coords.py

* FINALLY!!!!!Force Controller is working

* Cleaning up ForceController

* Created offsets and added more addons: ForceSensor and apply_force

File: robo_gym/data/ur5/ur5_2f.urdf (robot description, URDF)
Before this commit: robot ur5, 21 links, 20 joints
Links:
- removed link base
- added link left_sensor_pad, mass 0.0001; collision box size=0.001 0.017 0.035; visual box size=0.001 0.025 0.035
- added link right_sensor_pad, mass 0.0001; collision box size=0.001 0.017 0.035; visual box size=0.001 0.025 0.035
- link ee_link: geometry visual box size=0.01 0.01 0.01
- link left_finger_pad: mass None -> 0.001
- link right_finger_pad: mass None -> 0.001
Joints:
- removed joint base_link-base_fixed_joint
- added joint left_pad_sensor_joint: type fixed, parent left_finger_pad, child left_sensor_pad, origin xyz=0.0035 0 0.01 rpy=0 0 0
- added joint right_pad_sensor_joint: type fixed, parent right_finger_pad, child right_sensor_pad, origin xyz=0.0035 0 0.01 rpy=0 0 0
- joint ee_fixed_joint: origin xyz=0.0 0.0823 0.0 rpy=0.0 0.0 1.57079632679 -> xyz=0.0 0.241 0.0 rpy=0.0 0.0 0.0
